File: USBoard/elec/USBoard.kicad_pcb (KiCad board)
At the start: 2 copper layers, 45 x 34.8 mm, 44 parts, among them IC1 ATTINY45-P, P1 USB_OTG, P2 CONN_01X02, P3 USB_B, P4 CONN_02X06, P5 CONN_02X03, P6 CONN_01X06

Commit message: Add silk & properties
Parts:
- added REF***: OSHW-Logo2_7.3x6mm_SilkScreen, Symbols:OSHW-Logo2_7.3x6mm_SilkScreen, B.Cu at (140.2, 77.0)
- moved REF*** 21.7 mm to (139.7, 78.2)
Other:
- board text added: "http://u.dinask.eu/usb"
- board text added: "v1.0 GPLv3"
